Commit message: fixed args to spawn UR10 in a specific position, now the world_to_base_link joint is updated so that the tf tree is correct

File: ur_description/urdf/ur10_robot.urdf.xacro (robot description, xacro)
@@ -5,4 +5,10 @@
   <xacro:arg name="max_torque_scale_factor" default="1.0"/>
   <xacro:arg name="max_velocity_scale_factor" default="1.0"/>
+  <xacro:arg name="x" default="0.0"/>
+  <xacro:arg name="y" default="0.0"/>
+  <xacro:arg name="z" default="0.0"/>
+  <xacro:arg name="roll" default="0.0"/>
+  <xacro:arg name="pitch" default="0.0"/>
+  <xacro:arg name="yaw" default="0.0"/>
   <!-- common stuff -->
   <xacro:include filename="$(find ur_description)/urdf/common.gazebo.xacro" />
@@ -19,5 +25,5 @@
     <parent link="world" />
     <child link = "base_link" />
-    <origin xyz="0.0 0.0 0.0" rpy="0.0 0.0 0.0" />
+    <origin xyz="$(arg x) $(arg y) $(arg z)" rpy="$(arg roll) $(arg pitch) $(arg yaw)" />
   </joint>
 </robot>
